File: KiCad/WiC64_Plugin.kicad_pcb (KiCad board)
At the start: 2 copper layers, 54.4 x 63.7 mm, 59 parts, among them CN1 USERPORT-C64, Q1 BSS138, Q10 BSS138, Q11 BSS138, Q2 BSS138, Q3 BSS138, Q4 BSS138, Q5 BSS138, Q6 BSS138, Q7 BSS138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

Commit message: Find/Reconstruct missing libs/footprints and fix most DRC problems PCB is mostly untouched so far, focus was just on "completing" the released source files
Parts:
- C1, C2: footprint w_capacitors:CP_6.3x11mm_hor -> w_capacitors:CP_6.3x11mm_horiz-R
- H1, H2: renamed from REF**; value MountingHole_3.2mm_M3_ISO7380 -> MountingHole
- V1: renamed from G***; value LOGO -> GMP
- V2: renamed from G***; value LOGO -> YPS
- V3: renamed from G***; value LOGO -> LazyJones
- V4: renamed from G***; value LOGO -> KiWi
- V5: renamed from REF**; value ESD-Logo_6.6x6mm_SilkScreen -> ESD_WARN
- moved C1 6.53 mm to (145.8, 125.6)
- moved C2 6.48 mm to (164.0, 130.2)
- moved V3 0.38 mm to (149.7, 123.9)
- moved V4 0.32 mm to (162.9, 124.1)
Other:
- rule pad_to_mask_clearance: 0.051 -> 0
